File: noise_gate/noise_gate.kicad_pcb (KiCad board)
At the start: 2 copper layers, 80 x 100 mm, 71 parts, among them J1 Jack_6.35, J2 Jack_6.35, J3 Jack_6.35, J4 Jack_6.35, J6 top_panel_connector, J9 Barrel_Jack_Switch, P1 front_panel, P2 bottom_panel, Q1 MMBT5551, Q10 AO3401A, Q13 AO3400A, Q14 AO3400A, Q2 MMBT5551, Q3 MMBT5551, Q4 MMBT5551, Q5 MMBT5551, Q8 AO3401A, SW1 pedala_switch

Commit message: schematic done
Parts:
- removed C14, C16, C17: 10u, Capacitor_SMD:C_0603_1608Metric_Pad1.08x0.95mm_HandSolder
- removed C18, C4: 100n, Capacitor_SMD:C_0603_1608Metric_Pad1.08x0.95mm_HandSolder
- removed C19, C20: 470u, Capacitor_THT:CP_Radial_D8.0mm_P3.50mm
- removed C3, C6: 1u, Capacitor_SMD:C_0603_1608Metric_Pad1.08x0.95mm_HandSolder
- removed C5, C9: 470p, Capacitor_SMD:C_0603_1608Metric_Pad1.08x0.95mm_HandSolder
- removed D5: 1N4148WS, Diode_SMD:D_SOD-323
- removed Q1, Q2, Q4, Q5: MMBT5551, Package_TO_SOT_SMD:SOT-23
- removed Q10, Q8: AO3401A, Package_TO_SOT_SMD:SOT-23
- removed Q13, Q14: AO3400A, Package_TO_SOT_SMD:SOT-23
- removed R12: 10k, Resistor_SMD:R_0603_1608Metric_Pad0.98x0.95mm_HandSolder
- removed R21: 3.3k, Resistor_SMD:R_0603_1608Metric_Pad0.98x0.95mm_HandSolder
- added BT1: Battery_Cell, pedale:BatteryHolder_Eagle_12BH611-GR, F.Cu at (75.0, 94.1)
- added C15: 47n, Capacitor_SMD:C_0603_1608Metric_Pad1.08x0.95mm_HandSolder, F.Cu at (148.8, 28.1)
- added C25: 1u, Capacitor_SMD:C_0603_1608Metric_Pad1.08x0.95mm_HandSolder, F.Cu at (148.8, 38.1)
- added C26: 1n, Capacitor_SMD:C_0603_1608Metric_Pad1.08x0.95mm_HandSolder, F.Cu at (148.8, 40.6)
- added C28: 10u, Capacitor_SMD:C_0603_1608Metric_Pad1.08x0.95mm_HandSolder, F.Cu at (148.8, 43.1)
- added C29: 10u, Capacitor_SMD:C_0603_1608Metric_Pad1.08x0.95mm_HandSolder, F.Cu at (148.8, 45.7)
- added C30: 1u, Capacitor_SMD:C_0603_1608Metric_Pad1.08x0.95mm_HandSolder, F.Cu at (148.8, 48.2)
- added C31: 10u, Capacitor_SMD:C_0603_1608Metric_Pad1.08x0.95mm_HandSolder, F.Cu at (153.2, 28.1)
- added C32: 10u, Capacitor_SMD:C_0603_1608Metric_Pad1.08x0.95mm_HandSolder, F.Cu at (153.2, 30.6)
- added D8: M7, Diode_SMD:D_SMA, F.Cu at (169.2, 70.7)
- added J7: Conn_01x01_Socket, TestPoint:TestPoint_THTPad_D2.5mm_Drill1.2mm, F.Cu at (69.0, 94.0)
- added J8: Conn_01x01_Socket, TestPoint:TestPoint_THTPad_D2.5mm_Drill1.2mm, F.Cu at (68.9, 106.8)
- added JP1: SolderJumper_3_Bridged12, Jumper:SolderJumper-3_P1.3mm_Bridged12_Pad1.0x1.5mm, F.Cu at (166.9, 41.4)
- added Q11: MMBF5486, Package_TO_SOT_SMD:SOT-23, F.Cu at (144.2, 29.2)
- added Q12: MMBT5551, Package_TO_SOT_SMD:SOT-23, F.Cu at (144.2, 33.9)
- added Q15: MMBT5551, Package_TO_SOT_SMD:SOT-23, F.Cu at (144.2, 38.5)
- added Q16: MMBT5551, Package_TO_SOT_SMD:SOT-23, F.Cu at (144.2, 43.1)
- added Q17: MMBT5551, Package_TO_SOT_SMD:SOT-23, F.Cu at (144.2, 47.7)
- added Q18: MMBT5551, Package_TO_SOT_SMD:SOT-23, F.Cu at (144.2, 52.4)
- added R28: 1k, Resistor_SMD:R_0603_1608Metric_Pad0.98x0.95mm_HandSolder, F.Cu at (161.6, 82.0)
- added R35: 470k, Resistor_SMD:R_0603_1608Metric_Pad0.98x0.95mm_HandSolder, F.Cu at (153.2, 48.2)
- added R43: 47k, Resistor_SMD:R_0603_1608Metric_Pad0.98x0.95mm_HandSolder, F.Cu at (157.6, 28.1)
- added R44: 47k, Resistor_SMD:R_0603_1608Metric_Pad0.98x0.95mm_HandSolder, F.Cu at (157.6, 30.6)
- added R45: 100k, Resistor_SMD:R_0603_1608Metric_Pad0.98x0.95mm_HandSolder, F.Cu at (157.6, 33.1)
- added R46: 100k, Resistor_SMD:R_0603_1608Metric_Pad0.98x0.95mm_HandSolder, F.Cu at (157.6, 35.6)
- added R47: 470, Resistor_SMD:R_0603_1608Metric_Pad0.98x0.95mm_HandSolder, F.Cu at (157.6, 38.1)
- added R48: 4.7k, Resistor_SMD:R_0603_1608Metric_Pad0.98x0.95mm_HandSolder, F.Cu at (157.6, 40.6)
- added R49: 10k, Resistor_SMD:R_0603_1608Metric_Pad0.98x0.95mm_HandSolder, F.Cu at (157.6, 43.1)
- added R50: 33k, Resistor_SMD:R_0603_1608Metric_Pad0.98x0.95mm_HandSolder, F.Cu at (157.6, 45.7)
- added R51: 10k, Resistor_SMD:R_0603_1608Metric_Pad0.98x0.95mm_HandSolder, F.Cu at (157.6, 48.2)
- added R52: 100k, Resistor_SMD:R_0603_1608Metric_Pad0.98x0.95mm_HandSolder, F.Cu at (161.9, 28.1)
- added R53: 47k, Resistor_SMD:R_0603_1608Metric_Pad0.98x0.95mm_HandSolder, F.Cu at (161.9, 30.6)
- added R55: 10k, Resistor_SMD:R_0603_1608Metric_Pad0.98x0.95mm_HandSolder, F.Cu at (161.9, 35.6)
- added R57: 1k, Resistor_SMD:R_0603_1608Metric_Pad0.98x0.95mm_HandSolder, F.Cu at (161.9, 38.1)
- added RV2: 4.7k, Potentiometer_THT:Potentiometer_Bourns_3296W_Vertical, F.Cu at (172.2, 30.0)
- added RV5: 4.7k, Potentiometer_THT:Potentiometer_Bourns_3296W_Vertical, F.Cu at (172.2, 36.4)
- C1: value 470p -> 2.2u
- C10: value 100n -> 10u
- C11: value 100n -> 22nF
- C12: value 4.7n -> 1u
- C13: value 10n -> 33nF
- C2: value 1u -> 22nF
- R1: value 47k -> 1Meg
- R10, R15: value 10k -> 1Meg
- R11, R16: value 150 -> 10k
- R13: value 100k -> 1Meg
- R14: value 470k -> 3.3k
- R17: value 39k -> 470k
- R18: value 100k -> 4.7k
- R19: value 470k -> 220k
- R2: value 100 -> 22k
- R20: value 15k -> 680
- R22: value 22k -> 470
- R3: value 47k -> 22k
- R4: value 470k -> 22k
- R8: value 100k -> 68k
- moved C11 109.1 mm to (223.7, 67.8)
- moved D3 109.1 mm to (190.6, 80.6)
- moved R11 109.1 mm to (185.6, 83.3)
- moved R17 109.1 mm to (199.7, 69.3)
- moved R19 109.1 mm to (216.6, 67.3)
- moved R20 109.1 mm to (223.7, 71.7)
- moved R22 109.1 mm to (203.2, 69.4)
- moved R25 109.1 mm to (216.6, 56.4)
- moved R26 109.1 mm to (210.8, 76.7)
- moved R3 109.1 mm to (187.2, 72.5)
- moved R4 109.1 mm to (181.7, 68.4)
- moved R7 109.1 mm to (179.1, 77.3)
- moved R8 109.1 mm to (187.7, 78.0)
- moved R9 109.1 mm to (182.7, 79.9)
- moved C1 109.1 mm to (183.3, 68.4)
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Connections:
- C1 pad 1: Net-(Q4-B) -> Net-(Q11-D)
- C1 pad 2: Net-(Q4-C) -> Net-(Q3-B)
- C10 pad 1: F_OUT -> Net-(C10-Pad1)
- C10 pad 2: Net-(Q3-B) -> Net-(J6C-Pin_12)
- C11 pad 1: Net-(Q3-C) -> Net-(J6A-Pin_2)
- C11 pad 2: Net-(J6C-Pin_12) -> IN_BUFF
- C12 pad 1: Net-(D1-A) -> 0
- C12 pad 2: Net-(J6B-Pin_5) -> 4V7
- C13 pad 1: 0 -> Net-(C13-Pad1)
- C13 pad 2: Net-(J6B-Pin_9) -> Net-(Q3-E)
- C2 pad 2: Net-(Q4-B) -> /in+
- C7 pad 1: Net-(C7-Pad1) -> unconnected-(C7-Pad1)
- C7 pad 2: Net-(Q2-B) -> unconnected-(C7-Pad2)
- C8 pad 1: Net-(Q2-B) -> Net-(C8-Pad1)
- C8 pad 2: Net-(D1-K) -> Net-(Q3-B)
- D1 pad 2: Net-(D1-A) -> 0
- D2 pad 1: Net-(D1-A) -> Net-(D2-K)
- D2 pad 2: Net-(D1-K) -> 0
- D3 pad 1: Net-(D3-K) -> CONTROL
- J1 pad T: SW_IN -> Net-(J1-PadT)
- J2 pad T: Net-(SW1A-B) -> SEND_OUT
- J3 pad T: unconnected-(J3-PadT) -> Net-(SW1A-B)
- J4 pad S: unconnected-(J4-PadS) -> 0
- J4 pad T: unconnected-(J4-PadT) -> Net-(J4-PadT)
- J6 pad 2: FS_OUT -> Net-(J6A-Pin_2)
- J6 pad 5: Net-(J6B-Pin_5) -> CONTROL
- J6 pad 7: F_OUT -> Net-(J6B-Pin_7)
- J9 pad 1: CONN+ -> 0
- J9 pad 2: CONN- -> 9V
- J9 pad 3: BAT- -> BAT+
- Q3 pad 3: Net-(Q3-C) -> 9V
- R1 pad 1: Net-(Q4-B) -> /in+
- R1 pad 2: 0 -> 4.5V
- R10 pad 1: 9V -> Net-(Q11-G)
- R10 pad 2: Net-(D3-K) -> Net-(C13-Pad1)
- R11 pad 1: Net-(Q1-E) -> 0
- R11 pad 2: 0 -> Net-(C32-Pad1)
- R13 pad 1: Net-(Q2-B) -> Net-(Q11-G)
- R13 pad 2: 0 -> CONTROL
- R14 pad 1: Net-(Q2-B) -> 9V
- R14 pad 2: Net-(D1-A) -> 4V7
- R15 pad 2: Net-(D1-A) -> Net-(Q3-B)
- R16 pad 1: Net-(Q2-E) -> 0
- R16 pad 2: 0 -> Net-(Q3-E)
- R17 pad 1: Net-(D1-A) -> Net-(C26-Pad1)
- R17 pad 2: Net-(J6B-Pin_9) -> Net-(U1B--)
- R18 pad 1: Net-(Q3-B) -> 0
- R18 pad 2: 0 -> Net-(J6A-Pin_6)
- R19 pad 1: Net-(Q3-B) -> 4.5V
- R19 pad 2: 9V -> Net-(U1B-+)
- R2 pad 1: 0 -> 4.5V
- R2 pad 2: Net-(Q4-E) -> 9V
- R20 pad 1: Net-(Q3-C) -> Net-(C25-Pad2)
- R20 pad 2: 9V -> Net-(U1B--)
- R22 pad 1: 0 -> Net-(Q3-E)
- R22 pad 2: Net-(J6B-Pin_5) -> Net-(C10-Pad1)
- R24 pad 1: Net-(Q5-B) -> IN_BUFF
- R24 pad 2: REG_IN -> Net-(U1A--)
- R3 pad 1: SW_IN -> RETURN_BUFF
- R3 pad 2: Net-(C2-Pad1) -> Net-(C8-Pad1)
- R4 pad 1: Net-(Q4-B) -> 0
- R4 pad 2: Net-(Q4-C) -> 4.5V
- R5 pad 1: 9V -> Net-(C32-Pad1)
- R5 pad 2: Net-(Q4-C) -> IN_BUFF
- R6 pad 1: Net-(J6A-Pin_6) -> Net-(C2-Pad1)
- R6 pad 2: 0 -> Net-(J4-PadT)
- R7 pad 1: Net-(J6A-Pin_4) -> 0
- R7 pad 2: Net-(C4-Pad1) -> Net-(Q12-B)
- R8 pad 1: Net-(Q1-B) -> 4V7
- R8 pad 2: 0 -> Net-(Q12-B)
- R9 pad 1: Net-(Q1-B) -> 4V7
- R9 pad 2: Net-(D3-K) -> Net-(Q11-D)
- SW1 pad 1: SW_IN -> SEND_OUT
Routing:
- net 9V: track 213.1 -> 0.00 mm, vias 6 -> 0
- net SW_IN: track 95.5 -> 0.00 mm, vias 7 -> 0
- net Net-(J6C-Pin_14): track 75.8 -> 0.00 mm, vias 3 -> 0
- net Net-(SW1B-B): track 60.9 -> 0.00 mm
- net BAT-: track 59.7 -> 0.00 mm
- net unconnected-(J3-PadTN): track 53.5 -> 0.00 mm, vias 2 -> 0
- net REG_IN: track 48.9 -> 0.00 mm
- net Net-(J6D-Pin_8): track 36.3 -> 0.00 mm, vias 1 -> 0
- net (no net): track 33.3 -> 0.00 mm
- net Net-(J6A-Pin_4): track 31.0 -> 0.00 mm
- net CONN-: track 28.6 -> 0.00 mm
- net Net-(SW1A-B): track 28.3 -> 0.00 mm
- net Net-(J6C-Pin_12): track 25.6 -> 0.00 mm
- net CONN+: track 22.0 -> 0.00 mm, vias 1 -> 0
- net Net-(D1-A): track 22.0 -> 0.00 mm
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