File: noise_gate/noise_gate.kicad_pcb (KiCad board)
At the start: 2 copper layers, 80 x 100 mm, 85 parts, among them J1 Jack_6.35, J2 Jack_6.35, J3 Jack_6.35, J4 Jack_6.35, J6 top_panel_connector, J7 Conn_01x01_Socket, J8 Conn_01x01_Socket, J9 Barrel_Jack_Switch, P1 front_panel, P2 bottom_panel, Q11 MMBF5486, Q12 MMBT5551, Q15 MMBT5551, Q16 MMBT5551, Q17 MMBT5551, Q18 MMBT5551, Q3 MMBT5551, SW1 pedala_switch

Commit message: gruba postavka komponenta
Parts:
- removed C7: 100n, Capacitor_SMD:C_0603_1608Metric_Pad1.08x0.95mm_HandSolder
- added U1: TL072, Package_SO:SOIC-8_3.9x4.9mm_P1.27mm, F.Cu at (112.7, 56.3)
- moved R18 146.0 mm to (73.5, 51.8)
- moved R52 125.6 mm to (76.4, 120.1), turned to 180 degrees
- moved C10 121.7 mm to (98.2, 46.0), turned to 90 degrees
- moved R5 121.0 mm to (77.5, 126.5), turned to -90 degrees
- moved C32 119.6 mm to (76.6, 122.4), turned to 180 degrees
- moved R11 117.9 mm to (75.7, 126.3), turned to 90 degrees
- moved R26 117.9 mm to (101.7, 121.5)
- moved C11 115.8 mm to (108.0, 61.0), turned to 0 degrees
- moved R20 111.6 mm to (113.8, 51.8), turned to 180 degrees
- moved D8 104.4 mm to (69.1, 100.5), turned to -90 degrees
- moved R22 102.8 mm to (102.7, 48.0), turned to 90 degrees
- moved R19 101.3 mm to (116.3, 52.9), turned to -90 degrees
- moved R17 90.9 mm to (110.5, 51.7), turned to 0 degrees
- moved C31 82.4 mm to (186.1, 103.6), turned to 90 degrees
- moved R53 76.9 mm to (188.5, 102.7)
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Routing:
- net Net-(J6A-Pin_6): track 0.00 -> 12.8 mm
- net 0: vias 0 -> 1

Commit message: gotov layout!
Parts:
- added C33: 1u, Capacitor_SMD:C_0603_1608Metric_Pad1.08x0.95mm_HandSolder, F.Cu at (109.1, 54.3)
- JP1: moved to B.Cu
- moved R3 107.9 mm to (85.0, 77.2), turned to 90 degrees
- moved R55 104.7 mm to (86.5, 77.2), turned to 90 degrees
- moved R49 101.9 mm to (91.0, 71.4), turned to 90 degrees
- moved R53 101.5 mm to (89.0, 82.7), turned to 180 degrees
- moved Q18 99.0 mm to (89.2, 79.5), turned to -90 degrees
- moved R57 98.3 mm to (92.7, 83.0), turned to 180 degrees
- moved RV2 97.0 mm to (94.7, 70.7), turned to -90 degrees
- moved Q3 96.6 mm to (80.3, 77.7), turned to -90 degrees
- moved C28 96.1 mm to (100.2, 81.7)
- moved C31 96.1 mm to (92.6, 81.5), turned to 180 degrees
- moved R43 95.8 mm to (100.2, 83.3)
- moved JP1 95.8 mm to (88.8, 59.5), turned to 180 degrees
- moved R16 95.3 mm to (75.8, 80.0), turned to 90 degrees
- moved Q15 95.0 mm to (103.7, 80.9)
- moved R45 94.4 mm to (98.0, 78.3), turned to 180 degrees
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Routing:
- net 9V: track 0.00 -> 238.2 mm, vias 0 -> 11
- net IN_BUFF: track 0.00 -> 108.3 mm
- net Net-(J6D-Pin_8): track 0.00 -> 106.9 mm
- net Net-(J6C-Pin_14): track 0.00 -> 80.1 mm, vias 0 -> 2
- net 4.5V: track 0.00 -> 77.5 mm, vias 0 -> 6
- net CONTROL: track 0.00 -> 62.6 mm, vias 0 -> 1
- net BAT+: track 0.00 -> 59.5 mm
- net Net-(J6C-Pin_12): track 0.00 -> 55.6 mm
- net Net-(SW1A-B): track 0.00 -> 46.5 mm
- net Net-(J1-PadT): track 0.00 -> 43.3 mm, vias 0 -> 2
- net Net-(J6A-Pin_2): track 0.00 -> 36.9 mm, vias 0 -> 1
- net Net-(J6A-Pin_4): track 0.00 -> 35.5 mm, vias 0 -> 1
- net Net-(Q15-B): track 0.00 -> 28.0 mm
- net SEND_OUT: track 0.00 -> 23.4 mm
- net 0: track 0.00 -> 22.0 mm, vias 1 -> 40
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