File: noise_gate/noise_gate.kicad_sch (KiCad schematic)
At the start: 71 parts, among them J1 Jack_6.35, J2 Jack_6.35, J3 Jack_6.35, J4 Jack_6.35, J6 top_panel_connector, J9 Barrel_Jack_Switch, P1 front_panel, P2 bottom_panel, Q1 MMBT5551, Q10 AO3401A, Q13 AO3400A, Q14 AO3400A, Q2 MMBT5551, Q3 MMBT5551, Q4 MMBT5551, Q5 MMBT5551, Q8 AO3401A, SW1 pedala_switch

Commit message: sa
Parts:
- removed Q1, Q2, Q4: MMBT5551, Package_TO_SOT_SMD:SOT-23, symbol Transistor_BJT:BC817
- added C15: 47n, Capacitor_SMD:C_0603_1608Metric_Pad1.08x0.95mm_HandSolder, symbol Device:C
- added C21, C27: 100n, Capacitor_SMD:C_0603_1608Metric_Pad1.08x0.95mm_HandSolder, symbol Device:C
- added C22, C28, C29, C31, C32, C33: 10u, Capacitor_SMD:C_0603_1608Metric_Pad1.08x0.95mm_HandSolder, symbol Device:C
- added C23, C24: 220p, Capacitor_SMD:C_0603_1608Metric_Pad1.08x0.95mm_HandSolder, symbol Device:C
- added C25, C30: 1u, Capacitor_SMD:C_0603_1608Metric_Pad1.08x0.95mm_HandSolder, symbol Device:C
- added C26: 1n, Capacitor_SMD:C_0603_1608Metric_Pad1.08x0.95mm_HandSolder, symbol Device:C
- added D4: 1N4148WS, Diode_SMD:D_SOD-323, symbol Diode:1N4148WS
- added JP1: SolderJumper_3_Bridged12, Jumper:SolderJumper-3_P1.3mm_Bridged12_Pad1.0x1.5mm, symbol Jumper:SolderJumper_3_Bridged12
- added JP4: Jumper_2_Open, Jumper:SolderJumper-2_P1.3mm_Open_RoundedPad1.0x1.5mm, symbol Jumper:Jumper_2_Open
- added JP9: Jumper_2_Bridged, Jumper:SolderJumper-2_P1.3mm_Bridged_RoundedPad1.0x1.5mm, symbol Jumper:Jumper_2_Bridged
- added Q1, Q2, Q4, Q6: 2N7002, Package_TO_SOT_SMD:SOT-23, symbol Transistor_FET:2N7002
- added Q11: MMBF5486, Package_TO_SOT_SMD:SOT-23, symbol Transistor_FET:MMBF4392
- added Q12, Q15, Q16, Q17, Q18, Q7, Q9: MMBT5551, Package_TO_SOT_SMD:SOT-23, symbol Transistor_BJT:BC817
- added R23, R45, R46, R52, R54: 100k, Resistor_SMD:R_0603_1608Metric_Pad0.98x0.95mm_HandSolder, symbol Device:R
- added R27: 2.2k, Resistor_SMD:R_0603_1608Metric_Pad0.98x0.95mm_HandSolder, symbol Device:R
- added R28, R29, R30, R57: 1k, Resistor_SMD:R_0603_1608Metric_Pad0.98x0.95mm_HandSolder, symbol Device:R
- added R31, R32, R33, R36, R37, R38, R40, R41, R49, R51, R55: 10k, Resistor_SMD:R_0603_1608Metric_Pad0.98x0.95mm_HandSolder, symbol Device:R
- added R34: 20k, Resistor_SMD:R_0603_1608Metric_Pad0.98x0.95mm_HandSolder, symbol Device:R
- added R35: 470k, Resistor_SMD:R_0603_1608Metric_Pad0.98x0.95mm_HandSolder, symbol Device:R
- added R39, R42: 3.3k, Resistor_SMD:R_0603_1608Metric_Pad0.98x0.95mm_HandSolder, symbol Device:R
- added R43, R44, R53: 47k, Resistor_SMD:R_0603_1608Metric_Pad0.98x0.95mm_HandSolder, symbol Device:R
- added R47: 470, Resistor_SMD:R_0603_1608Metric_Pad0.98x0.95mm_HandSolder, symbol Device:R
- added R48: 4.7k, Resistor_SMD:R_0603_1608Metric_Pad0.98x0.95mm_HandSolder, symbol Device:R
- added R50: 33k, Resistor_SMD:R_0603_1608Metric_Pad0.98x0.95mm_HandSolder, symbol Device:R
- added RV1: 100k, symbol Device:R_Potentiometer
- added RV2, RV5: 4.7k, Potentiometer_THT:Potentiometer_Bourns_3296W_Vertical, symbol Device:R_Potentiometer
- added U1: TL072, symbol Amplifier_Operational:TL072
- added V1: VSIN, symbol Simulation_SPICE:VSIN
- added V2: 9, symbol Simulation_SPICE:VDC
- C1: value 470p -> 2.2u; LCSC C1620 -> C21122
- C10: value 100n -> 10u; LCSC C14663 -> C96446
- C11: value 100n -> 22nF; LCSC C14663 -> C21122
- C12: value 4.7n -> 1u; LCSC C53987 -> C15849
- C13: value 10n -> 33nF; LCSC C57112 -> C1614
- C2: value 1u -> 22nF; LCSC C15849 -> C21122
- C4: value 100n -> 1u; LCSC C14663 -> C15849
- C5: value 470p -> 1u; LCSC C1620 -> C15849
- C9: value 470p -> 47n; LCSC C1620 -> C1622
- J6: footprint pedale:IDC-Header_2x08_P2.54mm_Vertical -> Connector_IDC:IDC-Header_2x08_P2.54mm_Vertical
- R1: value 47k -> 1Meg
- R10, R15, R5: value 10k -> 1Meg; LCSC C25804 -> C25819
- R11: value 150 -> 100; LCSC C22808 -> C22775
- R12: value 10k -> 100; LCSC C25804 -> C22775
- R13: value 100k -> 1Meg; LCSC C25803 -> C25819
- R14: value 470k -> 3.3k; LCSC C23178 -> C22978
- R16: value 150 -> 10k; LCSC C22808 -> C25804
- R17: value 39k -> 100k; LCSC C23153 -> C25803
- R18: value 100k -> 4.7k; LCSC C25803 -> C23162
- R19: value 470k -> 220k; LCSC C23178 -> C22961
- R2: value 100 -> 47k; LCSC C22775 -> C25819
- R20: value 15k -> 680; LCSC C22809 -> C23228
- R21: value 3.3k -> 1Meg; LCSC C22978 -> C25819
- R22: value 22k -> 470; LCSC C31850 -> C23179
- R3: value 47k -> 22k; LCSC C25819 -> C31850
- R4: value 470k -> 47k; LCSC C23178 -> C25819
- R8: value 100k -> 68k; LCSC C25803 -> C23231
Connections:
- net 0: now also C12.1, D1.2 (A), D2.2 (A), J4.S, R16.1, R17.2, R18.1, R4.2, R7.1, C21.1, C22.2, C27.1, C30.1, Q12.2 (E), Q16.2 (E), Q17.2 (E), R23.2, R36.1, R38.1, R39.2, R41.1, R42.2, R44.2, R45.2, R46.2, R48.1, R49.1, R52.2, R54.2, R55.2, U1.4 (V-), V1.2, V2.2; no longer C13.1, R1.2, R11.2, R13.2, R16.2, R18.2, R2.1, R21.2, R22.1, R6.2, R8.2
- net 9V: now also Q3.3 (C), R14.1, R2.1, Q18.3 (C), Q7.3 (C), Q9.3 (C), R29.1, R37.2, R40.2, R43.1, U1.8 (V+), V2.1; no longer R10.1, R19.2, R20.2, R5.1
- net in+: now reaches C2.2, R1.1
- net in+: now also U1.3 (+); no longer C1.1, R4.1
- net at J6.4 (Pin_4): now also C15.1; no longer R7.1
- net at J6.6 (Pin_6): now also R18.2; no longer R6.1
- net at R11.1: now also C22.1
- net at C2.1: now also R6.1; no longer R3.2
- net at J2.T: now also C32.2, R52.1; no longer SW1.2 (B)
- net at Q3.2 (E): now also C13.2, R16.2, R22.1; no longer R21.1
- net 4.5V: now reaches R2.2
- net 4.5V: now also R1.2, R19.1, R4.1, R5.2, C25.1, R53.2
- net at J3.T: now also SW1.2 (B)
- net at R7.2: now also R8.2, Q12.1 (B); no longer C4.1
- net at R12.2: now also C23.1, R27.2; no longer C7.1
- net at J6.12 (Pin_12): no longer C11.2
- net at J4.T: now also R6.2, V1.1
- net FS_OUT: no longer names the net of J6.2 (Pin_2)
- net FS_OUT: now also C11.1; no longer C3.2
- net F_OUT: no longer names the net of C10.1
- net F_OUT: now also R22.2; no longer J6.7 (Pin_7)
- removed net SW_IN: J1.T, R3.1, SW1.1 (A)
- new net: C10.2, R17.1
- new net: R49.2, RV2.1
- new net: R51.2, RV2.2
- new net: R50.1, RV2.3, RV5.2
- new net: Q4.1 (G), Q6.1 (G), R30.1
- new net: Q4.2 (S), Q6.2 (S)
- new net: Q4.3 (D), Q9.2 (E), R42.1
- new net: C29.2, D1.1 (K), Q16.1 (B), R45.1
- new net: C4.1, JP9.1 (A), Q2.3 (D)
- new net: C5.1, JP9.2 (B), Q6.3 (D), R23.1
- new net: Q16.3 (C), Q17.3 (C), R47.1
- new net: Q11.3 (G), R10.1, R13.1
- new net: D5.1 (K), R31.2, R32.1
- new net: D4.1 (K), D5.2 (A)
- new net: C29.1, Q15.2 (E), R44.1
- new net: R48.2, RV5.1
- new net: C4.2, Q9.1 (B), R40.1, R41.2
- new net: C3.2, R31.1, R34.1
- new net: C13.1, R10.2
- new net: Q1.1 (G), Q2.1 (G), R28.1
- new net: Q1.2 (S), Q2.2 (S)
- new net: C5.2, Q7.1 (B), R36.2, R37.1
- new net: C6.1, Q7.2 (E), R39.1
- new net: C33.2, R54.1, SW1.1 (A)
- new net: C28.2, D2.1 (K), Q17.1 (B), R46.1
- new net: C28.1, Q15.3 (C), R43.2
- new net: J6.9 (Pin_9), JP1.1 (A), R50.2
- new net: C23.2, C24.1
- new net: C26.2, Q15.1 (B), R35.1
- new net: C9.2, R5.1
- new net: C15.2, R19.2, U1.5 (+)
- new net: R20.2, R21.1, U1.6 (-)
- new net: C26.1, R21.2, R35.2, U1.7
- new net: C8.1, R3.2
- new net: C1.2, C8.2, Q3.1 (B), R15.2
- new net: C31.2, Q18.1 (B), R53.1
- new net: C6.2, R38.2
- new net: J6.7 (Pin_7), JP1.2 (C)
- new net: C25.2, R20.1
- new net: C31.1, R57.1
- new net: J1.T, R57.2
- new net: R33.2, R34.2
- new net: R11.2, R12.1
- new net: D4.2 (A), R32.2, R33.1
- new net: C24.2, C3.1, RV1.2, RV1.3
- new net: R27.1, RV1.1
- new net: D3.2 (A), R51.1
- new net: C27.2, JP4.2 (B), R30.2
- new net: C1.1, Q11.1 (D), R9.2
- new net 4V7: C12.2, Q11.2 (S), Q12.3 (C), R14.2, R8.1, R9.1, RV5.3
- new net CONTROL: C30.2, D3.1 (K), J6.5 (Pin_5), JP1.3 (B), R13.2, R47.2
- new net INPUT_BUFFER: Q1.3 (D)
- new net IN_BUFF: C11.2, C32.1, C33.1, C9.1, U1.1, U1.2 (-)
- new net OUTPUT_ENABLE: C21.2, JP4.1 (A), R28.2, R29.2
- new net RETURN_BUFF: Q18.2 (E), R3.1, R55.1
- now unconnected: C7.2
- no-connect marks 19 -> 16
Other:
- note added: ".ic V(/in+)=4.5"
- note added: "100 KB"
- note added: "C23162"
- note added: "INPUT"
- note added: "OUTPUT"
- note added: "Peak detection"
- note added: "RETURN"
- note added: "SEND"
- note added: "Stopping stage"
- note added: "sensitivity"
- note removed: "Clipping and tone stage"
- note removed: "Output gain stage and selection switch"
- moved on the sheet: C14, C16, C17, C18, C19, C20, C7, D1, H1, H2, H3, H4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

Commit message: schematic done
Parts:
- removed C14, C16, C17, C22, C33: 10u, Capacitor_SMD:C_0603_1608Metric_Pad1.08x0.95mm_HandSolder, symbol Device:C
- removed C18, C21, C27: 100n, Capacitor_SMD:C_0603_1608Metric_Pad1.08x0.95mm_HandSolder, symbol Device:C
- removed C19, C20: 470u, Capacitor_THT:CP_Radial_D8.0mm_P3.50mm, symbol Device:C_Polarized_US
- removed C23, C24: 220p, Capacitor_SMD:C_0603_1608Metric_Pad1.08x0.95mm_HandSolder, symbol Device:C
- removed C3, C4, C5, C6: 1u, Capacitor_SMD:C_0603_1608Metric_Pad1.08x0.95mm_HandSolder, symbol Device:C
- removed C9: 47n, Capacitor_SMD:C_0603_1608Metric_Pad1.08x0.95mm_HandSolder, symbol Device:C
- removed D4, D5: 1N4148WS, Diode_SMD:D_SOD-323, symbol Diode:1N4148WS
- removed JP4: Jumper_2_Open, Jumper:SolderJumper-2_P1.3mm_Open_RoundedPad1.0x1.5mm, symbol Jumper:Jumper_2_Open
- removed JP9: Jumper_2_Bridged, Jumper:SolderJumper-2_P1.3mm_Bridged_RoundedPad1.0x1.5mm, symbol Jumper:Jumper_2_Bridged
- removed Q1, Q2, Q4, Q6: 2N7002, Package_TO_SOT_SMD:SOT-23, symbol Transistor_FET:2N7002
- removed Q10, Q8: AO3401A, Package_TO_SOT_SMD:SOT-23, symbol Transistor_FET:AO3401A
- removed Q13, Q14: AO3400A, Package_TO_SOT_SMD:SOT-23, symbol Transistor_FET:AO3400A
- removed Q5, Q7, Q9: MMBT5551, Package_TO_SOT_SMD:SOT-23, symbol Transistor_BJT:BC817
- removed R12: 100, Resistor_SMD:R_0603_1608Metric_Pad0.98x0.95mm_HandSolder, symbol Device:R
- removed R21: 1Meg, Resistor_SMD:R_0603_1608Metric_Pad0.98x0.95mm_HandSolder, symbol Device:R
- removed R23, R54: 100k, Resistor_SMD:R_0603_1608Metric_Pad0.98x0.95mm_HandSolder, symbol Device:R
- removed R27: 2.2k, Resistor_SMD:R_0603_1608Metric_Pad0.98x0.95mm_HandSolder, symbol Device:R
- removed R29, R30: 1k, Resistor_SMD:R_0603_1608Metric_Pad0.98x0.95mm_HandSolder, symbol Device:R
- removed R31, R32, R33, R36, R37, R38, R40, R41: 10k, Resistor_SMD:R_0603_1608Metric_Pad0.98x0.95mm_HandSolder, symbol Device:R
- removed R34: 20k, Resistor_SMD:R_0603_1608Metric_Pad0.98x0.95mm_HandSolder, symbol Device:R
- removed R39, R42: 3.3k, Resistor_SMD:R_0603_1608Metric_Pad0.98x0.95mm_HandSolder, symbol Device:R
- removed RV1: 100k, symbol Device:R_Potentiometer
- added BT1: Battery_Cell, pedale:BatteryHolder_Eagle_12BH611-GR, symbol Device:Battery_Cell
- added D8: M7, Diode_SMD:D_SMA, symbol Diode:MRA4005T3G
- added J7, J8: Conn_01x01_Socket, TestPoint:TestPoint_THTPad_D2.5mm_Drill1.2mm, symbol Connector:Conn_01x01_Socket
- R11: value 100 -> 10k; LCSC C22775 -> C25804
- R17: value 100k -> 470k; LCSC C25803 -> C23178
- R2, R4: value 47k -> 22k; LCSC C25819 -> C31850
- R5: value 1Meg -> 10k; LCSC C25819 -> C25804
Connections:
- net CONN+ is gone; now on net 0: J9.1
- net CONN- is gone; now on net 9V: J9.2
- net OUTPUT_ENABLE is gone; now on net 0: R28.2
- net REG_IN is gone; now on an unnamed net: R24.2
- net 0: now also R11.1, R4.1, D8.2 (A); no longer R17.2, R4.2
- net 4.5V: now also R2.1, R4.2; no longer R2.2, R4.1, R5.2
- net 9V: now also R2.2, D8.1 (K); no longer R2.1
- net BAT-: now also BT1.2 (-), J8.1 (Pin_1); no longer J9.3
- net IN_BUFF: now also R24.1, R5.2; no longer C32.1, U1.2 (-)
- net at C10.2: now also J6.12 (Pin_12); no longer R17.1
- net at R28.1: now also U1.2 (-)
- net SEND_OUT: now reaches C32.2, J2.T, R52.1
- net SEND_OUT: now also SW1.1 (A)
- net at R5.1: now also C32.1, R11.2
- net at R20.2, U1.6 (-): now also R17.2
- net at C26.1, R35.2, U1.7: now also R17.1
- new net BAT+: BT1.1 (+), J7.1 (Pin_1), J9.3
Other:
- note added: "Send"
- note removed: ".ic V(/in+)=4.5"
- note removed: "Power supply filtering"
- moved on the sheet: C1, C10, C12, C13, C31, C32, C8, H1, H2, H3, H4, H5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

Commit message: gruba postavka komponenta
Parts:
- removed C7: 100n, Capacitor_SMD:C_0603_1608Metric_Pad1.08x0.95mm_HandSolder, symbol Device:C
- U1: footprint (none) -> Package_SO:SOIC-8_3.9x4.9mm_P1.27mm
Other:
- moved on the sheet: D3
Changed lines of the file:
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@@
 	(wire
 		(pts
+			(xy 330.2 55.88) (xy 332.74 55.88)
+		)
+		(stroke
+			(width 0)
+			(type default)
+		)
+	)
+	(wire
+		(pts
 			(xy 163.83 135.89) (xy 163.83 132.08)
 		)
@@
 	(wire
 		(pts
-			(xy 332.74 55.88) (xy 328.93 55.88)
-		)
-		(stroke
-			(width 0)
-			(type default)
-		)
-	)
-	(wire
-		(pts
 			(xy 219.71 40.64) (xy 219.71 41.91)
 		)
@@
 	(wire
 		(pts
+			(xy 322.58 55.88) (xy 321.31 55.88)
+		)
+		(stroke
+			(width 0)
+			(type default)
+		)
+	)
+	(wire
+		(pts
 			(xy 218.44 133.35) (xy 223.52 133.35)
 		)
@@
 			)
 		)
-		(property "Footprint" ""
+		(property "Footprint" "Package_SO:SOIC-8_3.9x4.9mm_P1.27mm"
 			(at 77.47 218.44 0)
 			(effects
@@
 			)
 		)
-		(property "Footprint" ""
+		(property "Footprint" "Package_SO:SOIC-8_3.9x4.9mm_P1.27mm"
 			(at 175.26 49.53 0)
 			(effects
@@
 	)
 	(symbol
-		(lib_id "Device:C")
-		(at 49.53 71.12 90)
-		(unit 1)
-		(exclude_from_sim no)
-		(in_bom yes)
-		(on_board yes)
-		(dnp no)
-		(fields_autoplaced yes)
-		(property "Reference" "C7"
-			(at 49.53 63.5 90)
-			(effects
-				(font
-					(size 1.27 1.27)
-				)
-			)
-		)
-		(property "Value" "100n"
-			(at 49.53 66.04 90)
-			(effects
-				(font
-					(size 1.27 1.27)
-				)
-			)
-		)
-		(property "Footprint" "Capacitor_SMD:C_0603_1608Metric_Pad1.08x0.95mm_HandSolder"
-			(at 53.34 70.1548 0)
-			(effects
-				(font
-					(size 1.27 1.27)
-				)
-				(hide yes)
-			)
-		)
-		(property "Datasheet" "~"
-			(at 49.53 71.12 0)
-			(effects
-				(font
-					(size 1.27 1.27)
-				)
-				(hide yes)
-			)
-		)
-		(property "Description" ""
-			(at 49.53 71.12 0)
-			(effects
-				(font
-					(size 1.27 1.27)
-				)
-			)
-		)
-		(property "LCSC" "C14663"
-			(at 49.53 71.12 90)
-			(effects
-				(font
-					(size 1.27 1.27)
-				)
-				(hide yes)
-			)
-		)
-		(pin "1"
-		)
-		(pin "2"
-		)
-		(instances
-			(project "noise_gate"
-				(path "/1fda0e48-ac05-4486-b24b-352a2425b266"
-					(reference "C7")
-					(unit 1)
-				)
-			)
-		)
-	)
-	(symbol
 		(lib_id "Simulation_SPICE:0")
 		(at 179.07 140.97 0)
@@
 	(symbol
 		(lib_id "Diode:1N4148WS")
-		(at 325.12 55.88 0)
+		(at 326.39 55.88 0)
 		(mirror x)
 		(unit 1)
@@
 		(dnp no)
 		(property "Reference" "D3"
-			(at 330.2 58.42 0)
+			(at 331.47 58.42 0)
 			(effects
 				(font
@@
 		)
 		(property "Value" "1N4148WS"
-			(at 330.2 60.96 0)
+			(at 331.47 60.96 0)
 			(effects
 				(font
@@
 		)
 		(property "Footprint" "Diode_SMD:D_SOD-323"
-			(at 325.12 51.435 0)
+			(at 326.39 51.435 0)
 			(effects
 				(font
@@
 		)
 		(property "Datasheet" "https://www.vishay.com/docs/85751/1n4148ws.pdf"
-			(at 325.12 55.88 0)
+			(at 326.39 55.88 0)
 			(effects
 				(font
@@
 		)
 		(property "Description" ""
-			(at 325.12 55.88 0)
+			(at 326.39 55.88 0)
 			(effects
 				(font
@@
 		)
 		(property "Sim.Device" "D"
-			(at 325.12 55.88 0)
+			(at 326.39 55.88 0)
 			(effects
 				(font
@@
 		)
 		(property "Sim.Pins" "1=K 2=A"
-			(at 325.12 55.88 0)
+			(at 326.39 55.88 0)
 			(effects
 				(font
@@
 		)
 		(property "Sim.Library" "/home/ostoja/spice_models/diode/1N4148.lib"
-			(at 325.12 55.88 0)
+			(at 326.39 55.88 0)
 			(effects
 				(font
@@
 		)
 		(property "Sim.Name" "1N4148"
-			(at 325.12 55.88 0)
+			(at 326.39 55.88 0)
 			(effects
 				(font
@@
 		)
 		(property "LCSC" "C2128"
-			(at 325.12 55.88 0)
+			(at 326.39 55.88 0)
 			(effects
 				(font
@@
 		(on_board yes)
 		(dnp no)
-		(fields_autoplaced yes)
 		(property "Reference" "#GND016"
 			(at 73.66 280.67 0)
@@
 			)
 		)
-		(property "Footprint" ""
+		(property "Footprint" "Package_SO:SOIC-8_3.9x4.9mm_P1.27mm"
 			(at 82.55 49.53 0)
 			(effects
